Commit message: ros2エコシステムに合わせた修正

File: gng_vlut_system/urdf/topoarm_description/urdf/_topoarm.urdf.xacro (robot description, xacro)
@@ -2,5 +2,5 @@
 <robot xmlns:xacro="http://www.ros.org/wiki/xacro">
   <xacro:macro name="topoarm" params="prefix parent xyz rpy">
-    <xacro:property name="meshes_file_direction" value="package://topoarm_description/meshes/topoarm"/>
+    <xacro:property name="meshes_file_direction" value="package://gng_vlut_system/urdf/topoarm_description/meshes/topoarm"/>
     <joint name="${prefix}base_joint" type="fixed">
       <parent link="${parent}"/>

Commit message: ちらつきやや解消

File: gng_vlut_system/urdf/topoarm_description/urdf/_topoarm.urdf.xacro (robot description, xacro)
@@ -14,5 +14,5 @@
           <mesh filename="${meshes_file_direction}/link1.stl" scale="0.001 0.001 0.001"/>
         </geometry>
-        <material name="grey"/>
+        <material name="green"/>
       </visual>
       <collision>
@@ -42,5 +42,5 @@
           <mesh filename="${meshes_file_direction}/link2.stl" scale="0.001 0.001 0.001"/>
         </geometry>
-        <material name="grey"/>
+        <material name="green"/>
       </visual>
       <collision>
@@ -70,5 +70,5 @@
           <mesh filename="${meshes_file_direction}/link3.stl" scale="0.001 0.001 0.001"/>
         </geometry>
-        <material name="grey"/>
+        <material name="green"/>
       </visual>
       <collision>
@@ -98,5 +98,5 @@
           <mesh filename="${meshes_file_direction}/link4.stl" scale="0.001 0.001 0.001"/>
         </geometry>
-        <material name="grey"/>
+        <material name="green"/>
       </visual>
       <collision>
@@ -126,5 +126,5 @@
           <mesh filename="${meshes_file_direction}/link5.stl" scale="0.001 0.001 0.001"/>
         </geometry>
-        <material name="grey"/>
+        <material name="green"/>
       </visual>
       <collision>
@@ -154,5 +154,5 @@
           <mesh filename="${meshes_file_direction}/link6.stl" scale="0.001 0.001 0.001"/>
         </geometry>
-        <material name="grey"/>
+        <material name="green"/>
       </visual>
       <collision>
@@ -182,5 +182,5 @@
           <mesh filename="${meshes_file_direction}/link7.stl" scale="0.001 0.001 0.001"/>
         </geometry>
-        <material name="grey"/>
+        <material name="green"/>
       </visual>
       <collision>
@@ -202,5 +202,5 @@
           <mesh filename="${meshes_file_direction}/gripper_left_palm.stl" scale="0.001 0.001 0.001"/>
         </geometry>
-        <material name="grey"/>
+        <material name="green"/>
       </visual>
       <collision>
@@ -246,5 +246,5 @@
           <mesh filename="${meshes_file_direction}/gripper_right_palm.stl" scale="0.001 0.001 0.001"/>
         </geometry>
-        <material name="grey"/>
+        <material name="green"/>
       </visual>
       <collision>
@@ -271,5 +271,5 @@
           <box size="0.01 0.01 0.01" />
         </geometry>
-        <material name="grey"/>
+        <material name="green"/>
       </visual>
       <inertial>

File: gng_vlut_system/urdf/topoarm_description/urdf/topoarm_material.urdf.xacro (robot description, xacro)
@@ -2,5 +2,5 @@
 <robot xmlns:xacro="http://www.ros.org/wiki/xacro">
     <xacro:macro name="topoarm_material">
-        <material name="grey">
+        <material name="green">
         <color rgba="0.25 0.25 0.25 1.0"/>
         </material>

Commit message: 双腕召喚可能に変更

File: gng_vlut_system/urdf/topoarm_description/urdf/_topoarm.urdf.xacro (robot description, xacro)
@@ -228,7 +228,7 @@
     <joint name="${prefix}gripper_right_joint_mimic" type="fixed">
       <parent link="${prefix}link7" />
-      <child link="dummy_mimic_fix" />
-    </joint>
-    <link name="dummy_mimic_fix"/>
+      <child link="${prefix}dummy_mimic_fix" />
+    </joint>
+    <link name="${prefix}dummy_mimic_fix"/>
     <joint name="${prefix}gripper_right_joint" type="prismatic">
       <parent link="${prefix}link7"/>
