Commit message: 実機テスト追加？作業方針文書

File: urdf/topo_dual_arm_max/topo_dual_arm_max.urdf (robot description, URDF)
Before this commit: robot topo_dual_arm_max, 42 links, 41 joints
Links:
- link L_XM540_cover_link: geometry collision mesh filename=meshes/visual/urdf/XM540_cover.stl scale=0.001 0.001 0.001; visual mesh filename=meshes/visual/urdf/XM540_cover.stl scale=0.001 0.001 0.001
- link L_link4_cover_link: geometry collision mesh filename=meshes/visual/urdf/joint_cover.stl scale=0.001 0.001 0.001; visual mesh filename=meshes/visual/urdf/joint_cover.stl scale=0.001 0.001 0.001
- link L_link6_cover_link: geometry collision mesh filename=meshes/visual/urdf/joint_cover.stl scale=0.001 0.001 0.001; visual mesh filename=meshes/visual/urdf/joint_cover.stl scale=0.001 0.001 0.001
- link L_shoulder_cover_link: geometry collision mesh filename=meshes/visual/urdf/L_shoulder_cover.stl scale=0.001 0.001 0.001; visual mesh filename=meshes/visual/urdf/L_shoulder_cover.stl scale=0.001 0.001 0.001
- link R_XM540_cover_link: geometry collision mesh filename=meshes/visual/urdf/R_XM540_cover.stl scale=0.001 0.001 0.001; visual mesh filename=meshes/visual/urdf/R_XM540_cover.stl scale=0.001 0.001 0.001
- link R_link4_cover_link: geometry collision mesh filename=meshes/visual/urdf/joint_cover.stl scale=0.001 0.001 0.001; visual mesh filename=meshes/visual/urdf/joint_cover.stl scale=0.001 0.001 0.001
- link R_link6_cover_link: geometry collision mesh filename=meshes/visual/urdf/joint_cover.stl scale=0.001 0.001 0.001; visual mesh filename=meshes/visual/urdf/joint_cover.stl scale=0.001 0.001 0.001
- link R_shoulder_cover_link: geometry collision mesh filename=meshes/visual/urdf/shoulder_cover.stl scale=0.001 0.001 0.001; visual mesh filename=meshes/visual/urdf/shoulder_cover.stl scale=0.001 0.001 0.001
- link camera_link: geometry collision box size=0.025052487373352052 0.089856307983398442 0.025000000953674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; visual mesh filename=meshes/visual/urdf/realsense_camera.stl scale=0.001 0.001 0.001
- link neck_tilt_cover_link: geometry collision mesh filename=meshes/visual/urdf/joint_cover_cut.stl scale=0.001 0.001 0.001; visual mesh filename=meshes/visual/urdf/joint_cover_cut.stl scale=0.001 0.001 0.001
- link realsense_mount_link: geometry collision mesh filename=meshes/visual/urdf/realsense_mount.stl scale=0.001 0.001 0.001; visual mesh filename=meshes/visual/urdf/realsense_mount.stl scale=0.001 0.001 0.001
- link waist_cover_link: geometry collision mesh filename=meshes/visual/urdf/waist_cover.stl scale=0.001 0.001 0.001; visual mesh filename=meshes/visual/urdf/waist_cover.stl scale=0.001 0.001 0.001

File: urdf/topo_dual_arm_max_long/topo_dual_arm_max.urdf (robot description, URDF)
Before this commit: robot topo_dual_arm_max, 44 links, 43 joints
Links:
- link L_XM540_cover_link: geometry collision mesh filename=meshes/visual/urdf/XM540_cover.stl scale=0.001 0.001 0.001; visual mesh filename=meshes/visual/urdf/XM540_cover.stl scale=0.001 0.001 0.001
- link L_joint7_cover_link: geometry collision mesh filename=meshes/visual/urdf/joint_cover.stl scale=0.001 0.001 0.001; visual mesh filename=meshes/visual/urdf/joint_cover.stl scale=0.001 0.001 0.001
- link L_link4_cover_link: geometry collision mesh filename=meshes/visual/urdf/joint_cover.stl scale=0.001 0.001 0.001; visual mesh filename=meshes/visual/urdf/joint_cover.stl scale=0.001 0.001 0.001
- link L_link6_cover_link: geometry collision mesh filename=meshes/visual/urdf/joint_cover.stl scale=0.001 0.001 0.001; visual mesh filename=meshes/visual/urdf/joint_cover.stl scale=0.001 0.001 0.001
- link L_shoulder_cover_link: geometry collision mesh filename=meshes/visual/urdf/L_shoulder_cover.stl scale=0.001 0.001 0.001; visual mesh filename=meshes/visual/urdf/L_shoulder_cover.stl scale=0.001 0.001 0.001
- link R_XM540_cover_link: geometry collision mesh filename=meshes/visual/urdf/R_XM540_cover.stl scale=0.001 0.001 0.001; visual mesh filename=meshes/visual/urdf/R_XM540_cover.stl scale=0.001 0.001 0.001
- link R_joint7_cover_link: geometry collision mesh filename=meshes/visual/urdf/joint_cover.stl scale=0.001 0.001 0.001; visual mesh filename=meshes/visual/urdf/joint_cover.stl scale=0.001 0.001 0.001
- link R_link4_cover_link: geometry collision mesh filename=meshes/visual/urdf/joint_cover.stl scale=0.001 0.001 0.001; visual mesh filename=meshes/visual/urdf/joint_cover.stl scale=0.001 0.001 0.001
- link R_link6_cover_link: geometry collision mesh filename=meshes/visual/urdf/joint_cover.stl scale=0.001 0.001 0.001; visual mesh filename=meshes/visual/urdf/joint_cover.stl scale=0.001 0.001 0.001
- link R_shoulder_cover_link: geometry collision mesh filename=meshes/visual/urdf/shoulder_cover.stl scale=0.001 0.001 0.001; visual mesh filename=meshes/visual/urdf/shoulder_cover.stl scale=0.001 0.001 0.001
- link camera_link: geometry collision box size=0.025052487373352052 0.089856307983398442 0.025000000953674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; visual mesh filename=meshes/visual/urdf/realsense_camera.stl scale=0.001 0.001 0.001
- link neck_tilt_cover_link: geometry collision mesh filename=meshes/visual/urdf/joint_cover_cut.stl scale=0.001 0.001 0.001; visual mesh filename=meshes/visual/urdf/joint_cover_cut.stl scale=0.001 0.001 0.001
- link realsense_mount_link: geometry collision mesh filename=meshes/visual/urdf/realsense_mount.stl scale=0.001 0.001 0.001; visual mesh filename=meshes/visual/urdf/realsense_mount.stl scale=0.001 0.001 0.001
- link waist_cover_link: geometry collision mesh filename=meshes/visual/urdf/waist_cover.stl scale=0.001 0.001 0.001; visual mesh filename=meshes/visual/urdf/waist_cover.stl scale=0.001 0.001 0.001
