Commit message: 回避動作クオリティ改善必要。パラメータが多いきがする整理する必要がありそう

File: urdf/dual_arm_urdf/dual_arm_robot.urdf (robot description, URDF)
Before this commit: robot dual_arm_robot, 31 links, 30 joints
Links:
- link camera_link: geometry collision box size=0.025052487373352052 0.089856307983398442 0.025000000953674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; visual mesh filename=meshes/camera_link.stl scale=0.001 0.001 0.001
