Commit message: topofuzzyviewerの部品をurdfシミュレータの方に転用

File: ToPoDualArmMax_SourceDelivery_20260928/ToPoDualArmMax-Simulator/app/source.urdf (robot description, URDF)
Before this commit: robot topo_dual_arm_max, 44 links, 43 joints
Links:
- added link chest_lidar_link; collision box size=0.065033845603 0.072896927595 0.060257099569; visual mesh filename=meshes/chest_lidar_color_0.stl scale=0.001 0.001 0.001
- added link chest_lidar_mount_link; collision mesh filename=meshes/chest_lidar_mount_45.stl scale=0.001 0.001 0.001; visual mesh filename=meshes/chest_lidar_mount_45.stl scale=0.001 0.001 0.001
Joints:
- added joint chest_lidar_fixed: type fixed, parent chest_lidar_mount_link, child chest_lidar_link, origin xyz=0.041326157159 0 0.018326157159 rpy=0 0.785398163397 0
- added joint chest_lidar_mount_fixed: type fixed, parent torso_link, child chest_lidar_mount_link, origin xyz=0.028 0 0.102521097973 rpy=0 0 0

File: urdf/topo_dual_arm_max_long/topo_dual_arm_max.urdf (robot description, URDF)
Before this commit: robot topo_dual_arm_max, 44 links, 43 joints
Links:
- added link chest_lidar_link; collision box size=0.065033845603 0.072896927595 0.060257099569; visual mesh filename=meshes/chest_lidar_color_0.stl scale=0.001 0.001 0.001
- added link chest_lidar_mount_link; collision mesh filename=meshes/chest_lidar_mount_45.stl scale=0.001 0.001 0.001; visual mesh filename=meshes/chest_lidar_mount_45.stl scale=0.001 0.001 0.001
Joints:
- added joint chest_lidar_fixed: type fixed, parent chest_lidar_mount_link, child chest_lidar_link, origin xyz=0.041326157159 0 0.018326157159 rpy=0 0.785398163397 0
- added joint chest_lidar_mount_fixed: type fixed, parent torso_link, child chest_lidar_mount_link, origin xyz=0.028 0 0.102521097973 rpy=0 0 0

Commit message: base_footprintではなくbaselinkで一本化

File: ToPoDualArmMax_SourceDelivery_20260928/ToPoDualArmMax-Simulator/app/source.urdf (robot description, URDF)
Before this commit: robot topo_dual_arm_max, 46 links, 45 joints
Links:
- removed link base_footprint
Joints:
- removed joint base_footprint_to_base

File: urdf/topo_dual_arm_max_long/topo_dual_arm_max.urdf (robot description, URDF)
Before this commit: robot topo_dual_arm_max, 46 links, 45 joints
Links:
- removed link base_footprint
Joints:
- removed joint base_footprint_to_base
